File: boost.kicad_sch (KiCad schematic)
At the start: 25 parts, among them J2 Conn_01x10_Pin, J3 Conn_01x10_Pin, Q1 G1003B-23, U2 LM3478MA

Commit message: Switched to breadboard formfactor
Also added files for GH
Parts:
- removed H1, H2, H3, H4: MountingHole, MountingHole:MountingHole_3.2mm_M3, symbol Mechanical:MountingHole
- removed J2, J3: Conn_01x10_Pin, Connector_IDC:IDC-Header_2x05_P2.54mm_Vertical, symbol Connector:Conn_01x10_Pin
- removed JP2: Jumper_2_Small_Bridged, Connector_PinHeader_2.54mm:PinHeader_1x02_P2.54mm_Vertical_SMD_Pin1Left, symbol Jumper:Jumper_2_Small_Bridged
- removed TP1: TestPoint, CustomFootprints:TestPoint_Keystone_5019_Miniature, symbol Connector:TestPoint
- added J1, J4, J5, J6: Conn_01x01_Pin, Connector_PinHeader_2.54mm:PinHeader_1x01_P2.54mm_Vertical, symbol Connector:Conn_01x01_Pin
Connections:
- net GND: now also J4.1 (Pin_1), J6.1 (Pin_1)
- net 50V_BOOST renamed +50V
- net +50V: now also J5.1 (Pin_1)
- net VBUS renamed +5V
- net +5V: now also J1.1 (Pin_1)
Other:
- note added: "BOOST (50V)"
- note removed: "BOOST 1 (50V)"
- note removed: "From microcontroller board"
- note removed: "MOUTNING HOLES"
- note removed: "To nixie board"
- moved on the sheet: C10, C6, C7, C8, C9, D2, L1, Q1, R2, R3, R4, R5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

Commit message: Added calculators
Changed component values to match calculator recommended values
Parts:
- C10: value 120p -> 100p; LCSC PART # C18438 -> C7503509
- C9: value 120p -> 82p; LCSC PART # C18438 -> C1864236
- R4: value 390 -> 422; LCSC PART # C49653317 -> C5204003
- R6: value 150m -> 140m; LCSC PART # C37936 -> C37935
Other:
- note added: "Crossover: 5140 Hz PM: 79.3° Crossover Slope: -20.07 dB/dec"
- note added: "Python calculators included in the project repo were used for component selection. Peak switch current: 0.4A The mosfet, inductor, and diode should be able to handle this current * 1.5 (>0.6A) Output capacitor needs to be low ESR and needs to be rated for atleast 60V Output voltage is NOT variable, the potentiometer is only for callibration Use temperature stable and +-1% components where possible"
- note removed: "Crossover: 4760Hz PM: 77° Crossover Slope: -20.4 dB/dec"
- note removed: "Python calculators included in the project repo were used for component selection. Peak switch current: 0.4A The mosfet, inductor, and diode should be able to handle this current * 1.5 (>0.6A) Output capacitor needs to be low ESR and needs to be rated for atleast 60V Output voltage is NOT variable, the potentiometer is only for callibration"
- title: Power Supply Schematic -> Boost Converter Dev Board
Changed lines of the file:
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@@
 	(paper "A4")
 	(title_block
-		(title "Power Supply Schematic")
-		(date "2024-06-06")
-		(rev "0.1.1")
+		(title "Boost Converter Dev Board")
+		(date "2025-11-27")
+		(rev "1")
 	)
 	(rectangle
@@
 		)
 	)
-	(text "Python calculators included in the\nproject repo were used for component selection.\n\nPeak switch current: 0.4A\nThe mosfet, inductor, and diode should be\nable to handle this current * 1.5 (>0.6A)\n\nOutput capacitor needs to be low ESR and needs to be rated for atleast 60V\n\nOutput voltage is NOT variable, the potentiometer is only for callibration"
+	(text "Python calculators included in the\nproject repo were used for component selection.\n\nPeak switch current: 0.4A\nThe mosfet, inductor, and diode should be\nable to handle this current * 1.5 (>0.6A)\n\nOutput capacitor needs to be low ESR and needs to be rated for atleast 60V\n\nOutput voltage is NOT variable, the potentiometer is only for callibration\n\nUse temperature stable and +-1% components where possible"
 		(exclude_from_sim no)
-		(at 17.526 54.356 0)
+		(at 17.526 56.134 0)
 		(effects
 			(font
@@
 		)
 	)
-	(text "Crossover: 4760Hz\nPM: 77°\nCrossover Slope: -20.4 dB/dec"
+	(text "Crossover: 5140 Hz\nPM: 79.3°\nCrossover Slope: -20.07 dB/dec"
 		(exclude_from_sim no)
 		(at 87.122 139.446 0)
@@
 			)
 		)
-		(property "Value" "120p"
+		(property "Value" "82p"
 			(at 100.33 109.2199 0)
 			(effects
@@
 			)
 		)
-		(property "Datasheet" "https://www.lcsc.com/datasheet/C18438.pdf"
+		(property "Datasheet" "https://www.lcsc.com/datasheet/C1864236.pdf"
 			(at 96.52 107.95 0)
 			(effects
@@
 			)
 		)
-		(property "LCSC PART #" "C18438"
+		(property "LCSC PART #" "C1864236"
 			(at 96.52 107.95 0)
 			(effects
@@
 			)
 		)
-		(property "Value" "120p"
+		(property "Value" "100p"
 			(at 138.43 114.2999 0)
 			(effects
@@
 			)
 		)
-		(property "Datasheet" "https://www.lcsc.com/datasheet/C18438.pdf"
+		(property "Datasheet" "https://www.lcsc.com/datasheet/C7503509.pdf"
 			(at 134.62 113.03 0)
 			(effects
@@
 			)
 		)
-		(property "LCSC PART #" "C18438"
+		(property "LCSC PART #" "C7503509"
 			(at 134.62 113.03 0)
 			(effects
@@
 			)
 		)
-		(property "Value" "390"
+		(property "Value" "422"
 			(at 146.05 98.806 90)
 			(effects
@@
 			)
 		)
-		(property "Datasheet" "https://www.lcsc.com/datasheet/C49653317.pdf"
+		(property "Datasheet" "https://www.lcsc.com/datasheet/C5204003.pdf"
 			(at 146.05 101.6 0)
 			(effects
@@
 			)
 		)
-		(property "LCSC PART #" "C49653317"
+		(property "LCSC PART #" "C5204003"
 			(at 146.05 101.6 0)
 			(effects
@@
 			)
 		)
-		(property "Value" "150m"
+		(property "Value" "140m"
 			(at 161.29 118.1099 0)
 			(effects
@@
 			)
 		)
-		(property "Datasheet" "https://www.lcsc.com/datasheet/C37936.pdf"
+		(property "Datasheet" "https://www.lcsc.com/datasheet/C37935.pdf"
 			(at 158.75 116.84 0)
 			(effects
@@
 			)
 		)
-		(property "LCSC PART #" "C37936"
+		(property "LCSC PART #" "C37935"
 			(at 158.75 116.84 0)
 			(effects

Commit message: Changed to THT cap
Low ESR THT caps are easier to find. But I'm really changing cause the
SMD cap I wanted went out of stock :(
Parts:
- C6, C8: footprint Capacitor_SMD:CP_Elec_6.3x9.9 -> Capacitor_THT:CP_Radial_D6.3mm_P2.50mm; LCSC PART # C19270543 -> C44606504
Other:
- note added: "Crossover: 5140 Hz Phase margin: 78.46° Crossover Slope: -20.09 dB/dec Gain Margin: 23.61 dB"
- note removed: "Crossover: 5140 Hz PM: 79.3° Crossover Slope: -20.07 dB/dec"
Changed lines of the file:
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@@
 	(title_block
 		(title "Boost Converter Dev Board")
-		(date "2025-11-27")
-		(rev "1")
+		(date "2025-11-28")
+		(rev "2")
 	)
 	(rectangle
@@
 		)
 	)
-	(text "Crossover: 5140 Hz\nPM: 79.3°\nCrossover Slope: -20.07 dB/dec"
+	(text "Crossover: 5140 Hz\nPhase margin: 78.46°\nCrossover Slope: -20.09 dB/dec\nGain Margin: 23.61 dB"
 		(exclude_from_sim no)
 		(at 87.122 139.446 0)
@@
 			)
 		)
-		(property "Footprint" "Capacitor_SMD:CP_Elec_6.3x9.9"
+		(property "Footprint" "Capacitor_THT:CP_Radial_D6.3mm_P2.50mm"
 			(at 101.2952 81.28 0)
 			(effects
@@
 			)
 		)
-		(property "Datasheet" "https://www.lcsc.com/datasheet/C19270543.pdf"
+		(property "Datasheet" "https://www.lcsc.com/datasheet/C44606504.pdf"
 			(at 100.33 77.47 0)
 			(effects
@@
 			)
 		)
-		(property "LCSC PART #" "C19270543"
+		(property "LCSC PART #" "C44606504"
 			(at 100.33 77.47 0)
 			(effects
@@
 			)
 		)
-		(property "Footprint" "Capacitor_SMD:CP_Elec_6.3x9.9"
+		(property "Footprint" "Capacitor_THT:CP_Radial_D6.3mm_P2.50mm"
 			(at 202.8952 85.09 0)
 			(effects
@@
 			)
 		)
-		(property "Datasheet" "https://www.lcsc.com/datasheet/C19270543.pdf"
+		(property "Datasheet" "https://www.lcsc.com/datasheet/C44606504.pdf"
 			(at 201.93 81.28 0)
 			(effects
@@
 			)
 		)
-		(property "LCSC PART #" "C19270543"
+		(property "LCSC PART #" "C44606504"
 			(at 201.93 81.28 0)
 			(effects
